Commit message: update fsm, usd, task

File: grc26_isaacsim_task/assets/table.urdf (robot description, URDF)
Before this commit: robot pick_place_table, 9 links, 8 joints
Links:
- link table_top: mass 62.72000000000002 -> 117.60000000000001; geometry collision box size=2.0 1.2 0.07; visual box size=2.0 1.2 0.07
Joints:
- joint kinova1_table_mount_joint: origin xyz=-0.72 0.0 0.013 rpy=0 0 0 -> xyz=-0.915 0.0 0.013 rpy=0 0 0
- joint kinova2_table_mount_joint: origin xyz=0.72 0 0.013 rpy=0 0 0 -> xyz=0.915 0.0 0.013 rpy=0 0 0
- joint table_leg_bl_joint: origin xyz=-0.775 0.375 0.67 rpy=0 0 0 -> xyz=-0.975 0.575 0.67 rpy=0 0 0
- joint table_leg_br_joint: origin xyz=-0.775 -0.375 0.67 rpy=0 0 0 -> xyz=-0.975 -0.575 0.67 rpy=0 0 0
- joint table_leg_fl_joint: origin xyz=0.775 0.375 0.67 rpy=0 0 0 -> xyz=0.975 0.575 0.67 rpy=0 0 0
- joint table_leg_fr_joint: origin xyz=0.775 -0.375 0.67 rpy=0 0 0 -> xyz=0.975 -0.575 0.67 rpy=0 0 0
