Commit message: extend table length and minor fixes

File: grc26_kinova_moveit_config/config/pick_place.urdf (robot description, URDF)
Before this commit: robot gen3_2f_85_pick_place, 53 links, 52 joints
Links:
- link table_base: mass None -> 0.001
- link table_leg_bl: mass None -> 13.065000000000003
- link table_leg_br: mass None -> 13.065000000000003
- link table_leg_fl: mass None -> 13.065000000000003
- link table_leg_fr: mass None -> 13.065000000000003
- link table_top: mass None -> 117.60000000000001; geometry collision box size=2.0 1.2 0.07; visual box size=2.0 1.2 0.07
Joints:
- joint kinova1_base_joint: origin xyz=0 0 0.013 rpy=0 0 0 -> xyz=0 0 0.013 rpy=0 0 0.0
- joint kinova1_table_mount_joint: origin xyz=-0.7200000000000001 0 0.013 rpy=0 0 0 -> xyz=-0.915 0.0 0.013 rpy=0 0 0
- joint kinova2_base_joint: origin xyz=0 0 0.013 rpy=0 0 3.14159265359 -> xyz=0 0 0.013 rpy=0 0 -3.14159265359
- joint kinova2_table_mount_joint: origin xyz=0.7200000000000001 0 0.013 rpy=0 0 0 -> xyz=0.915 0.0 0.013 rpy=0 0 0
- joint table_leg_bl_joint: origin xyz=-0.775 0.375 0.67 rpy=0 0 0 -> xyz=-0.975 0.575 0.67 rpy=0 0 0
- joint table_leg_br_joint: origin xyz=-0.775 -0.375 0.67 rpy=0 0 0 -> xyz=-0.975 -0.575 0.67 rpy=0 0 0
- joint table_leg_fl_joint: origin xyz=0.775 0.375 0.67 rpy=0 0 0 -> xyz=0.975 0.575 0.67 rpy=0 0 0
- joint table_leg_fr_joint: origin xyz=0.775 -0.375 0.67 rpy=0 0 0 -> xyz=0.975 -0.575 0.67 rpy=0 0 0
